File: KiCad/macropad/macropad.kicad_sch (KiCad schematic)
At the start: 1 part

Commit message: Initial wiring
Parts:
- added J1: Conn_01x06, Connector_PinHeader_2.54mm:PinHeader_1x06_P2.54mm_Vertical, symbol Connector_Generic:Conn_01x06
- added LED1, LED2, LED3, LED4, LED5, LED6: LED_RGBA, Library:1.5mmRGBALED, symbol Device:LED_RGBA
- added R1, R2, R3, R4, R5, R6: 100, Resistor_SMD:R_0402_1005Metric, symbol Device:R
- added SW1, SW2, SW3, SW4, SW5, SW6: SW_DIP_x01, Library:SW_Cherry_MX_1.00u_PCB_LEDHole, symbol Switch:SW_DIP_x01
- U1: renamed from U?; footprint RPi_Pico:RPi_Pico_SMD_TH -> Pi-Pico:RPi_Pico_SMD
Connections:
- net 3V3: now also J1.6 (Pin_6), R1.1, R2.1, R3.1, R4.1, R5.1, R6.1
- net BTN1: now also SW1.2
- net BTN2: now also SW2.2
- net BTN3: now also SW3.2
- net BTN4: now also SW4.2
- net BTN5: now also U1.29 (GPIO22), SW5.2; no longer U1.21 (GPIO16)
- net BTN6: now also U1.24 (GPIO18), SW6.2; no longer U1.26 (GPIO20)
- net GND: now also J1.4 (Pin_4), SW1.1, SW2.1, SW3.1, SW4.1, SW5.1, SW6.1
- net LED1B: now also LED1.3 (BK)
- net LED1G: now also LED1.2 (GK)
- net LED1R: now also LED1.1 (RK)
- net LED2B: now also LED2.3 (BK)
- net LED2G: now also LED2.2 (GK)
- net LED2R: now also LED2.1 (RK)
- net LED3B: now also LED3.3 (BK)
- net LED3G: now also LED3.2 (GK)
- net LED3R: now also LED3.1 (RK)
- net LED4B: now also LED4.3 (BK)
- net LED4G: now also LED4.2 (GK)
- net LED4R: now also LED4.1 (RK)
- net LED5B: now also U1.34 (GPIO28_ADC2), LED5.3 (BK); no longer U1.25 (GPIO19)
- net LED5G: now also U1.32 (GPIO27_ADC1), LED5.2 (GK); no longer U1.24 (GPIO18)
- net LED5R: now also U1.31 (GPIO26_ADC0), LED5.1 (RK); no longer U1.22 (GPIO17)
- net LED6B: now also U1.27 (GPIO21), LED6.3 (BK); no longer U1.31 (GPIO26_ADC0)
- net LED6G: now also U1.26 (GPIO20), LED6.2 (GK); no longer U1.29 (GPIO22)
- net LED6R: now also U1.25 (GPIO19), LED6.1 (RK); no longer U1.27 (GPIO21)
- new net: LED3.4 (A), R3.2
- new net: LED1.4 (A), R1.2
- new net: LED4.4 (A), R4.2
- new net: LED6.4 (A), R6.2
- new net: LED5.4 (A), R5.2
- new net: LED2.4 (A), R2.2
- new net 3V3o: J1.5 (Pin_5)
- new net RST: J1.3 (Pin_3)
- new net SCL: J1.2 (Pin_2), U1.22 (GPIO17)
- new net SDA: J1.1 (Pin_1), U1.21 (GPIO16)

Commit message: Settings for gerber export
Parts:
- R1, R2, R3, R4, R5, R6: LCSC (none) -> C25076
Changed lines of the file:
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@@
+      (effects (font (size 1.27 1.27)) hide)
+    )
+    (property "LCSC" "C25076" (id 4) (at 48.26 93.98 90)
       (effects (font (size 1.27 1.27)) hide)
     )
@@
       (effects (font (size 1.27 1.27)) hide)
     )
+    (property "LCSC" "C25076" (id 4) (at 48.26 63.5 90)
+      (effects (font (size 1.27 1.27)) hide)
+    )
     (pin "1")
     (pin "2")
@@
       (effects (font (size 1.27 1.27)) hide)
     )
+    (property "LCSC" "C25076" (id 4) (at 48.26 109.22 90)
+      (effects (font (size 1.27 1.27)) hide)
+    )
     (pin "1")
     (pin "2")
@@
     )
     (property "Datasheet" "~" (id 3) (at 180.34 95.25 0)
+      (effects (font (size 1.27 1.27)) hide)
+    )
+    (property "LCSC" "C25076" (id 4) (at 180.34 95.25 90)
       (effects (font (size 1.27 1.27)) hide)
     )
@@
       (effects (font (size 1.27 1.27)) hide)
     )
+    (property "LCSC" "C25076" (id 4) (at 180.34 110.49 90)
+      (effects (font (size 1.27 1.27)) hide)
+    )
     (pin "1")
     (pin "2")
@@
       (effects (font (size 1.27 1.27)) hide)
     )
+    (property "LCSC" "C25076" (id 4) (at 48.26 78.74 90)
+      (effects (font (size 1.27 1.27)) hide)
+    )

Commit message: Use THT resistors, correct Kailh key layout, giving up on this project for now in favor of streamdekc
Parts:
- R1, R2, R3, R4, R5, R6: footprint Resistor_SMD:R_0402_1005Metric -> Resistor_THT:R_Axial_DIN0309_L9.0mm_D3.2mm_P12.70mm_Horizontal
- SW1, SW2, SW3, SW4, SW5, SW6: footprint Library:SW_Cherry_MX_1.00u_PCB_LEDHole -> Kailh Socket PG1350:Kailh_socket_PG1350
Changed lines of the file:
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@@
     (property "Reference" "SW4" (id 0) (at 93.98 96.3635 0))
     (property "Value" "SW_DIP_x01" (id 1) (at 93.98 99.1386 0))
-    (property "Footprint" "Library:SW_Cherry_MX_1.00u_PCB_LEDHole" (id 2) (at 93.98 102.87 0)
+    (property "Footprint" "Kailh Socket PG1350:Kailh_socket_PG1350" (id 2) (at 93.98 102.87 0)
       (effects (font (size 1.27 1.27)) hide)
     )
@@
     (property "Reference" "SW6" (id 0) (at 228.6 93.8235 0))
     (property "Value" "SW_DIP_x01" (id 1) (at 228.6 96.5986 0))
-    (property "Footprint" "Library:SW_Cherry_MX_1.00u_PCB_LEDHole" (id 2) (at 228.6 100.33 0)
+    (property "Footprint" "Kailh Socket PG1350:Kailh_socket_PG1350" (id 2) (at 228.6 100.33 0)
       (effects (font (size 1.27 1.27)) hide)
     )
@@
     (property "Reference" "SW2" (id 0) (at 93.98 70.9635 0))
     (property "Value" "SW_DIP_x01" (id 1) (at 93.98 73.7386 0))
-    (property "Footprint" "Library:SW_Cherry_MX_1.00u_PCB_LEDHole" (id 2) (at 93.98 77.47 0)
+    (property "Footprint" "Kailh Socket PG1350:Kailh_socket_PG1350" (id 2) (at 93.98 77.47 0)
       (effects (font (size 1.27 1.27)) hide)
     )
@@
     (property "Reference" "SW1" (id 0) (at 93.98 58.2635 0))
     (property "Value" "SW_DIP_x01" (id 1) (at 93.98 61.0386 0))
-    (property "Footprint" "Library:SW_Cherry_MX_1.00u_PCB_LEDHole" (id 2) (at 93.98 64.77 0)
+    (property "Footprint" "Kailh Socket PG1350:Kailh_socket_PG1350" (id 2) (at 93.98 64.77 0)
       (effects (font (size 1.27 1.27)) hide)
     )
@@
     (property "Reference" "R3" (id 0) (at 48.26 88.9975 90))
     (property "Value" "100" (id 1) (at 48.26 91.7726 90))
-    (property "Footprint" "Resistor_SMD:R_0402_1005Metric" (id 2) (at 48.26 95.758 90)
+    (property "Footprint" "Resistor_THT:R_Axial_DIN0309_L9.0mm_D3.2mm_P12.70mm_Horizontal" (id 2) (at 48.26 95.758 90)
       (effects (font (size 1.27 1.27)) hide)
     )
@@
     (property "Reference" "SW3" (id 0) (at 93.98 83.6635 0))
     (property "Value" "SW_DIP_x01" (id 1) (at 93.98 86.4386 0))
-    (property "Footprint" "Library:SW_Cherry_MX_1.00u_PCB_LEDHole" (id 2) (at 93.98 90.17 0)
+    (property "Footprint" "Kailh Socket PG1350:Kailh_socket_PG1350" (id 2) (at 93.98 90.17 0)
       (effects (font (size 1.27 1.27)) hide)
     )
@@
     (property "Reference" "R1" (id 0) (at 48.26 58.5175 90))
     (property "Value" "100" (id 1) (at 48.26 61.2926 90))
-    (property "Footprint" "Resistor_SMD:R_0402_1005Metric" (id 2) (at 48.26 65.278 90)
+    (property "Footprint" "Resistor_THT:R_Axial_DIN0309_L9.0mm_D3.2mm_P12.70mm_Horizontal" (id 2) (at 48.26 65.278 90)
       (effects (font (size 1.27 1.27)) hide)
     )
@@
     (property "Reference" "R4" (id 0) (at 48.26 104.2375 90))
     (property "Value" "100" (id 1) (at 48.26 107.0126 90))
-    (property "Footprint" "Resistor_SMD:R_0402_1005Metric" (id 2) (at 48.26 110.998 90)
+    (property "Footprint" "Resistor_THT:R_Axial_DIN0309_L9.0mm_D3.2mm_P12.70mm_Horizontal" (id 2) (at 48.26 110.998 90)
       (effects (font (size 1.27 1.27)) hide)
     )
@@
     (property "Reference" "R6" (id 0) (at 180.34 90.2675 90))
     (property "Value" "100" (id 1) (at 180.34 93.0426 90))
-    (property "Footprint" "Resistor_SMD:R_0402_1005Metric" (id 2) (at 180.34 97.028 90)
+    (property "Footprint" "Resistor_THT:R_Axial_DIN0309_L9.0mm_D3.2mm_P12.70mm_Horizontal" (id 2) (at 180.34 97.028 90)
       (effects (font (size 1.27 1.27)) hide)
     )
@@
     (property "Reference" "R5" (id 0) (at 180.34 105.5075 90))
     (property "Value" "100" (id 1) (at 180.34 108.2826 90))
-    (property "Footprint" "Resistor_SMD:R_0402_1005Metric" (id 2) (at 180.34 112.268 90)
+    (property "Footprint" "Resistor_THT:R_Axial_DIN0309_L9.0mm_D3.2mm_P12.70mm_Horizontal" (id 2) (at 180.34 112.268 90)
       (effects (font (size 1.27 1.27)) hide)
     )
@@
     (property "Reference" "SW5" (id 0) (at 228.6 106.5235 0))
     (property "Value" "SW_DIP_x01" (id 1) (at 228.6 109.2986 0))
-    (property "Footprint" "Library:SW_Cherry_MX_1.00u_PCB_LEDHole" (id 2) (at 228.6 113.03 0)
+    (property "Footprint" "Kailh Socket PG1350:Kailh_socket_PG1350" (id 2) (at 228.6 113.03 0)
       (effects (font (size 1.27 1.27)) hide)
     )
@@
     (property "Reference" "R2" (id 0) (at 48.26 73.7575 90))
     (property "Value" "100" (id 1) (at 48.26 76.5326 90))
-    (property "Footprint" "Resistor_SMD:R_0402_1005Metric" (id 2) (at 48.26 80.518 90)
+    (property "Footprint" "Resistor_THT:R_Axial_DIN0309_L9.0mm_D3.2mm_P12.70mm_Horizontal" (id 2) (at 48.26 80.518 90)
       (effects (font (size 1.27 1.27)) hide)
     )
@@
     )
     (path "/70f7cc60-4cd8-475f-9c30-b9ac53128161"
-      (reference "R1") (unit 1) (value "100") (footprint "Resistor_SMD:R_0402_1005Metric")
+      (reference "R1") (unit 1) (value "100") (footprint "Resistor_THT:R_Axial_DIN0309_L9.0mm_D3.2mm_P12.70mm_Horizontal")
     )
     (path "/f2e1c40f-3b6f-494f-bd3d-a67b8831428e"
-      (reference "R2") (unit 1) (value "100") (footprint "Resistor_SMD:R_0402_1005Metric")
+      (reference "R2") (unit 1) (value "100") (footprint "Resistor_THT:R_Axial_DIN0309_L9.0mm_D3.2mm_P12.70mm_Horizontal")
     )
     (path "/50725948-a952-443f-b645-c9aceffb3379"
-      (reference "R3") (unit 1) (value "100") (footprint "Resistor_SMD:R_0402_1005Metric")
+      (reference "R3") (unit 1) (value "100") (footprint "Resistor_THT:R_Axial_DIN0309_L9.0mm_D3.2mm_P12.70mm_Horizontal")
     )
     (path "/7302daac-ca55-40a6-9281-f06ebfbfccb9"
-      (reference "R4") (unit 1) (value "100") (footprint "Resistor_SMD:R_0402_1005Metric")
+      (reference "R4") (unit 1) (value "100") (footprint "Resistor_THT:R_Axial_DIN0309_L9.0mm_D3.2mm_P12.70mm_Horizontal")
     )
     (path "/d5bd8c39-c140-47ee-a4d9-49cb9ba225eb"
-      (reference "R5") (unit 1) (value "100") (footprint "Resistor_SMD:R_0402_1005Metric")
+      (reference "R5") (unit 1) (value "100") (footprint "Resistor_THT:R_Axial_DIN0309_L9.0mm_D3.2mm_P12.70mm_Horizontal")
     )
     (path "/a8c47e74-8b0b-426d-973d-34e5fea7e311"
-      (reference "R6") (unit 1) (value "100") (footprint "Resistor_SMD:R_0402_1005Metric")
+      (reference "R6") (unit 1) (value "100") (footprint "Resistor_THT:R_Axial_DIN0309_L9.0mm_D3.2mm_P12.70mm_Horizontal")
     )
     (path "/4b9676e0-276f-412c-afb1-51539cb10a75"
-      (reference "SW1") (unit 1) (value "SW_DIP_x01") (footprint "Library:SW_Cherry_MX_1.00u_PCB_LEDHole")
+      (reference "SW1") (unit 1) (value "SW_DIP_x01") (footprint "Kailh Socket PG1350:Kailh_socket_PG1350")
     )
     (path "/46a41e8b-8385-4e9f-9f62-dff54a2718bc"
-      (reference "SW2") (unit 1) (value "SW_DIP_x01") (footprint "Library:SW_Cherry_MX_1.00u_PCB_LEDHole")
+      (reference "SW2") (unit 1) (value "SW_DIP_x01") (footprint "Kailh Socket PG1350:Kailh_socket_PG1350")
     )
     (path "/5983fdbf-6097-455f-8e68-625e2c6dcc8e"
-      (reference "SW3") (unit 1) (value "SW_DIP_x01") (footprint "Library:SW_Cherry_MX_1.00u_PCB_LEDHole")
+      (reference "SW3") (unit 1) (value "SW_DIP_x01") (footprint "Kailh Socket PG1350:Kailh_socket_PG1350")
     )
     (path "/1106ee1e-05a7-4396-bcb7-ca7ab2b70d54"
-      (reference "SW4") (unit 1) (value "SW_DIP_x01") (footprint "Library:SW_Cherry_MX_1.00u_PCB_LEDHole")
+      (reference "SW4") (unit 1) (value "SW_DIP_x01") (footprint "Kailh Socket PG1350:Kailh_socket_PG1350")
     )
     (path "/db5f82fa-c141-47ed-8efa-a272eddf0110"
-      (reference "SW5") (unit 1) (value "SW_DIP_x01") (footprint "Library:SW_Cherry_MX_1.00u_PCB_LEDHole")
+      (reference "SW5") (unit 1) (value "SW_DIP_x01") (footprint "Kailh Socket PG1350:Kailh_socket_PG1350")
     )
     (path "/39d0fbd5-e5ed-4632-b96b-3041e65b0d99"
-      (reference "SW6") (unit 1) (value "SW_DIP_x01") (footprint "Library:SW_Cherry_MX_1.00u_PCB_LEDHole")
+      (reference "SW6") (unit 1) (value "SW_DIP_x01") (footprint "Kailh Socket PG1350:Kailh_socket_PG1350")
     )
     (path "/c10ace36-a93c-4c08-ac75-059ef9e1f71c"
